File: pyCopter_board/pycopter_board_v1.sch (EAGLE design)
At the start: 36 parts, among them Q1 32.768kHz, U1 BNO055, U3 BMP180

Commit message: Updated board
Parts:
- removed ESC1, ESC2, ESC3, ESC4: (no value), SparkFun-Connectors:M02PTH
- added JP1, JP2, JP3, JP4: (no value), SparkFun-Connectors:M03PTH
Connections:
- net GND: now also JP1.1, JP2.1, JP3.1, JP4.1; no longer ESC1.1, ESC2.1, ESC3.1, ESC4.1
- net P19: now also JP1.3; no longer ESC1.2
- net P20: now also JP3.3; no longer ESC2.2
- net P22: now also JP4.3; no longer ESC4.2
- net P23: now also JP2.3; no longer ESC3.2
- net VIN: now also JP1.2
Changed lines of the file:
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@@
 <part name="H7" library="holes" deviceset="MOUNT-HOLE" device="3.0"/>
 <part name="H8" library="holes" deviceset="MOUNT-HOLE" device="3.0"/>
-<part name="ESC1" library="SparkFun-Connectors" deviceset="M02" device="PTH"/>
-<part name="ESC2" library="SparkFun-Connectors" deviceset="M02" device="PTH"/>
-<part name="ESC3" library="SparkFun-Connectors" deviceset="M02" device="PTH"/>
-<part name="ESC4" library="SparkFun-Connectors" deviceset="M02" device="PTH"/>
+<part name="JP1" library="SparkFun-Connectors" deviceset="M03" device="PTH"/>
+<part name="JP2" library="SparkFun-Connectors" deviceset="M03" device="PTH"/>
+<part name="JP3" library="SparkFun-Connectors" deviceset="M03" device="PTH"/>
+<part name="JP4" library="SparkFun-Connectors" deviceset="M03" device="PTH"/>
 </parts>
 <sheets>
@@
 <instance part="GPSLEFT" gate="G$1" x="124.46" y="48.26"/>
 <instance part="GPSRIGHT" gate="G$1" x="165.1" y="43.18" rot="R180"/>
-<instance part="J3" gate="J$1" x="91.44" y="-22.86" rot="R90"/>
-<instance part="J4" gate="J$1" x="91.44" y="-7.62" rot="R90"/>
-<instance part="J5" gate="J$1" x="91.44" y="-38.1" rot="R90"/>
-<instance part="J6" gate="J$1" x="109.22" y="-38.1" rot="R90"/>
-<instance part="J7" gate="J$1" x="109.22" y="-22.86" rot="R90"/>
-<instance part="J8" gate="J$1" x="109.22" y="-7.62" rot="R90"/>
+<instance part="J3" gate="G$1" x="91.44" y="-22.86" rot="R90"/>
+<instance part="J4" gate="G$1" x="91.44" y="-7.62" rot="R90"/>
+<instance part="J5" gate="G$1" x="91.44" y="-38.1" rot="R90"/>
+<instance part="J6" gate="G$1" x="109.22" y="-38.1" rot="R90"/>
+<instance part="J7" gate="G$1" x="109.22" y="-22.86" rot="R90"/>
+<instance part="J8" gate="G$1" x="109.22" y="-7.62" rot="R90"/>
 <instance part="IMUBREAK" gate="G$1" x="180.34" y="-7.62"/>
 <instance part="BMP180BREAK" gate="G$1" x="139.7" y="-7.62"/>
@@
 <instance part="H7" gate="G$1" x="-99.06" y="60.96"/>
 <instance part="H8" gate="G$1" x="-93.98" y="50.8"/>
-<instance part="ESC1" gate="G$1" x="175.26" y="-25.4"/>
-<instance part="ESC2" gate="G$1" x="175.26" y="-38.1"/>
-<instance part="ESC3" gate="G$1" x="193.04" y="-25.4"/>
-<instance part="ESC4" gate="G$1" x="193.04" y="-38.1"/>
+<instance part="JP1" gate="G$1" x="177.8" y="-50.8"/>
+<instance part="JP2" gate="G$1" x="200.66" y="-50.8"/>
+<instance part="JP3" gate="G$1" x="177.8" y="-63.5"/>
+<instance part="JP4" gate="G$1" x="200.66" y="-63.5"/>
 </instances>
 <busses>
@@
 <wire x1="86.36" y1="63.5" x2="78.74" y2="63.5" width="0.1524" layer="91"/>
 <label x="78.74" y="63.5" size="1.778" layer="95"/>
+</segment>
+<segment>
+<pinref part="JP1" gate="G$1" pin="2"/>
+<wire x1="185.42" y1="-50.8" x2="190.5" y2="-50.8" width="0.1524" layer="91"/>
+<label x="190.5" y="-50.8" size="1.778" layer="95"/>
 </segment>
 </net>
@@
 </segment>
 <segment>
-<pinref part="J3" gate="J$1" pin="3"/>
+<pinref part="J3" gate="G$1" pin="3"/>
 <wire x1="88.9" y1="-15.24" x2="88.9" y2="-12.7" width="0.1524" layer="91"/>
 <label x="86.36" y="-15.24" size="1.778" layer="95"/>
@@
 </segment>
 <segment>
-<pinref part="ESC2" gate="G$1" pin="1"/>
-<wire x1="182.88" y1="-38.1" x2="185.42" y2="-38.1" width="0.1524" layer="91"/>
-<label x="185.42" y="-38.1" size="1.778" layer="95"/>
-</segment>
-<segment>
-<pinref part="ESC4" gate="G$1" pin="1"/>
-<wire x1="200.66" y1="-38.1" x2="203.2" y2="-38.1" width="0.1524" layer="91"/>
-<label x="203.2" y="-38.1" size="1.778" layer="95"/>
-</segment>
-<segment>
-<pinref part="ESC3" gate="G$1" pin="1"/>
-<wire x1="200.66" y1="-25.4" x2="205.74" y2="-25.4" width="0.1524" layer="91"/>
-<label x="205.74" y="-25.4" size="1.778" layer="95"/>
-</segment>
-<segment>
-<pinref part="ESC1" gate="G$1" pin="1"/>
-<wire x1="182.88" y1="-25.4" x2="185.42" y2="-25.4" width="0.1524" layer="91"/>
-<label x="185.42" y="-25.4" size="1.778" layer="95"/>
+<pinref part="JP3" gate="G$1" pin="1"/>
+<wire x1="185.42" y1="-66.04" x2="190.5" y2="-66.04" width="0.1524" layer="91"/>
+<label x="190.5" y="-66.04" size="1.778" layer="95"/>
+</segment>
+<segment>
+<pinref part="JP4" gate="G$1" pin="1"/>
+<wire x1="208.28" y1="-66.04" x2="213.36" y2="-66.04" width="0.1524" layer="91"/>
+<label x="213.36" y="-66.04" size="1.778" layer="95"/>
+</segment>
+<segment>
+<pinref part="JP2" gate="G$1" pin="1"/>
+<wire x1="208.28" y1="-53.34" x2="213.36" y2="-53.34" width="0.1524" layer="91"/>
+<label x="213.36" y="-53.34" size="1.778" layer="95"/>
+</segment>
+<segment>
+<pinref part="JP1" gate="G$1" pin="1"/>
+<wire x1="185.42" y1="-53.34" x2="190.5" y2="-53.34" width="0.1524" layer="91"/>
+<label x="190.5" y="-53.34" size="1.778" layer="95"/>
 </segment>
 </net>
@@
 </segment>
 <segment>
-<pinref part="J3" gate="J$1" pin="2"/>
+<pinref part="J3" gate="G$1" pin="2"/>
 <wire x1="91.44" y1="-15.24" x2="91.44" y2="-12.7" width="0.1524" layer="91"/>
 <label x="88.9" y="-12.7" size="1.778" layer="95"/>
@@
 <net name="THRO" class="0">
 <segment>
-<pinref part="J3" gate="J$1" pin="1"/>
+<pinref part="J3" gate="G$1" pin="1"/>
 <wire x1="93.98" y1="-15.24" x2="93.98" y2="-12.7" width="0.1524" layer="91"/>
 <label x="93.98" y="-15.24" size="1.778" layer="95"/>
@@
 <net name="ELEV" class="0">
 <segment>
-<pinref part="J5" gate="J$1" pin="1"/>
+<pinref part="J5" gate="G$1" pin="1"/>
 <wire x1="93.98" y1="-30.48" x2="93.98" y2="-27.94" width="0.1524" layer="91"/>
 <label x="93.98" y="-27.94" size="1.778" layer="95"/>
@@
 <net name="RUDD" class="0">
 <segment>
-<pinref part="J6" gate="J$1" pin="1"/>
+<pinref part="J6" gate="G$1" pin="1"/>
 <wire x1="111.76" y1="-30.48" x2="111.76" y2="-27.94" width="0.1524" layer="91"/>
 <label x="111.76" y="-27.94" size="1.778" layer="95"/>
@@
 <net name="GEAR" class="0">
 <segment>
-<pinref part="J7" gate="J$1" pin="1"/>
+<pinref part="J7" gate="G$1" pin="1"/>
 <wire x1="111.76" y1="-15.24" x2="111.76" y2="-12.7" width="0.1524" layer="91"/>
 <label x="111.76" y="-12.7" size="1.778" layer="95"/>
@@
 <net name="AUX1" class="0">
 <segment>
-<pinref part="J8" gate="J$1" pin="1"/>
+<pinref part="J8" gate="G$1" pin="1"/>
 <wire x1="111.76" y1="0" x2="111.76" y2="2.54" width="0.1524" layer="91"/>
 <label x="111.76" y="2.54" size="1.778" layer="95"/>
@@
 <net name="AILE" class="0">
 <segment>
-<pinref part="J4" gate="J$1" pin="1"/>
+<pinref part="J4" gate="G$1" pin="1"/>
 <wire x1="93.98" y1="0" x2="93.98" y2="2.54" width="0.1524" layer="91"/>
 <label x="96.52" y="2.54" size="1.778" layer="95"/>
@@
 </segment>
 <segment>
-<pinref part="ESC3" gate="G$1" pin="2"/>
-<wire x1="200.66" y1="-22.86" x2="205.74" y2="-22.86" width="0.1524" layer="91"/>
-<label x="205.74" y="-20.32" size="1.778" layer="95"/>
+<pinref part="JP2" gate="G$1" pin="3"/>
+<wire x1="208.28" y1="-48.26" x2="213.36" y2="-48.26" width="0.1524" layer="91"/>
+<label x="213.36" y="-48.26" size="1.778" layer="95"/>
 </segment>
 </net>
@@
 </segment>
 <segment>
-<pinref part="ESC4" gate="G$1" pin="2"/>
-<wire x1="200.66" y1="-35.56" x2="203.2" y2="-35.56" width="0.1524" layer="91"/>
-<label x="203.2" y="-35.56" size="1.778" layer="95"/>
+<pinref part="JP4" gate="G$1" pin="3"/>
+<wire x1="208.28" y1="-60.96" x2="213.36" y2="-60.96" width="0.1524" layer="91"/>
+<label x="213.36" y="-60.96" size="1.778" layer="95"/>
 </segment>
 </net>
@@
 </segment>
 <segment>
-<pinref part="ESC2" gate="G$1" pin="2"/>
-<wire x1="182.88" y1="-35.56" x2="185.42" y2="-35.56" width="0.1524" layer="91"/>
-<label x="185.42" y="-35.56" size="1.778" layer="95"/>
+<pinref part="JP3" gate="G$1" pin="3"/>
+<wire x1="185.42" y1="-60.96" x2="190.5" y2="-60.96" width="0.1524" layer="91"/>
+<label x="190.5" y="-60.96" size="1.778" layer="95"/>
 </segment>
 </net>
@@
 </segment>
 <segment>
-<pinref part="ESC1" gate="G$1" pin="2"/>
-<wire x1="182.88" y1="-22.86" x2="185.42" y2="-22.86" width="0.1524" layer="91"/>
-<label x="185.42" y="-22.86" size="1.778" layer="95"/>
-</segment>
-</net>
+<pinref part="JP1" gate="G$1" pin="3"/>
+<wire x1="185.42" y1="-48.26" x2="190.5" y2="-48.26" width="0.1524" layer="91"/>
+<label x="190.5" y="-48.26" size="1.778" layer="95"/>
+</segment>
+</net>
