File: pyCopter_board/pycopter_board_v1.sch (EAGLE design)
At the start: 36 parts, among them Q1 32.768kHz, U1 BNO055, U3 BMP180

Commit message: added some more updates based upon charlie's suggestions.
Parts:
- Q1: device special:XTAL/S -> crystal:CRYSTALTC38H
- R5, R6: value 10K -> 2.2k
Other:
- note removed: "Maybe an LED or 2? Also buttons?"
- note removed: "Need to decide what other LoPy pins should be exposed"
- note removed: "Not sure about I2C or UART connections for LoPy, or what pins will be used for servo signals."
- moved on the sheet: H5, H6, H8
