File: pyCopter_board/pycopter_board_v1.brd (EAGLE design)
At the start: 81 x 80 mm, 36 parts, among them Q1 32.768kHz, U1 BNO055, U3 BMP180

Commit message: Updated board
Parts:
- removed ESC1, ESC2, ESC3, ESC4: (no value), SparkFun-Connectors:1X02
- added JP1, JP2, JP3, JP4: (no value), SparkFun-Connectors:1X03
Connections:
- net GND: now also JP1.1, JP2.1, JP3.1, JP4.1; no longer ESC1.1, ESC2.1, ESC3.1, ESC4.1
- net P19: now also JP1.3; no longer ESC1.2
- net P20: now also JP3.3; no longer ESC2.2
- net P22: now also JP4.3; no longer ESC4.2
- net P23: now also JP2.3; no longer ESC3.2
- net VIN: now also JP1.2
Routing:
- net GND: track 396.6 -> 0.00 mm
- net 3.3V: track 254.3 -> 0.00 mm, vias 4 -> 0
- net SCL: track 152.0 -> 0.00 mm, vias 3 -> 0
- net P23: track 121.4 -> 0.00 mm, vias 1 -> 0
- net P19: track 114.5 -> 0.00 mm, vias 1 -> 0
- net SDA: track 113.3 -> 0.00 mm, vias 3 -> 0
- net P22: track 105.1 -> 0.00 mm, vias 1 -> 0
- net GPS_RX: track 80.3 -> 0.00 mm, vias 1 -> 0
- net GPS_TX: track 79.4 -> 0.00 mm
- net GEAR: track 74.3 -> 0.00 mm, vias 1 -> 0
- net RUDD: track 70.7 -> 0.00 mm
- net P20: track 60.1 -> 0.00 mm
- net THRO: track 54.9 -> 0.00 mm
- net AUX1: track 54.2 -> 0.00 mm
- net P17: track 53.6 -> 0.00 mm
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
Commit message: Added pycopter logo pictures
Routing:
- net GND: track 0.00 -> 389.1 mm, vias 0 -> 1
- net 3.3V: track 0.00 -> 242.6 mm, vias 0 -> 1
- net RUDD: track 0.00 -> 120.1 mm, vias 0 -> 2
- net SDA: track 0.00 -> 118.6 mm, vias 0 -> 2
- net P22: track 0.00 -> 112.4 mm
- net SCL: track 0.00 -> 111.6 mm, vias 0 -> 3
- net P23: track 0.00 -> 98.8 mm, vias 0 -> 2
- net GPS_RX: track 0.00 -> 83.7 mm, vias 0 -> 1
- net GEAR: track 0.00 -> 66.6 mm, vias 0 -> 2
- net P19: track 0.00 -> 63.9 mm
- net GPS_TX: track 0.00 -> 62.1 mm, vias 0 -> 1
- net P20: track 0.00 -> 49.0 mm
- net AUX1: track 0.00 -> 47.5 mm
- net XOUT: track 0.00 -> 47.4 mm, vias 0 -> 3
- net VIN: track 0.00 -> 45.3 mm
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